Commit message: done

File: urdf/gripper.xacro (robot description, xacro)
@@ -14,5 +14,5 @@
       <origin rpy="0 0 0" xyz="0 0 0"/>
       <geometry>
-        <mesh filename="package://project_final_mantzakidis_131/meshes/l_finger.dae"/>
+        <mesh filename="package://robot_project/meshes/l_finger.dae"/>
       </geometry>
     </visual>
@@ -34,5 +34,5 @@
       <origin rpy="0 0 0" xyz="0.09137 0.00495 0"/>
       <geometry>
-        <mesh filename="package://project_final_mantzakidis_131/meshes/l_finger_tip.dae"/>
+        <mesh filename="package://robot_project/meshes/l_finger_tip.dae"/>
       </geometry>
     </visual>
@@ -57,5 +57,5 @@
       <origin rpy="3.1415 0 0" xyz="0 0 0"/>
       <geometry>
-        <mesh filename="package://project_final_mantzakidis_131/meshes/l_finger.dae"/>
+        <mesh filename="package://robot_project/meshes/l_finger.dae"/>
       </geometry>
     </visual>
@@ -77,5 +77,5 @@
       <origin rpy="-3.1415 0 0" xyz="0.09137 0.00495 0"/>
       <geometry>
-        <mesh filename="package://project_final_mantzakidis_131/meshes/l_finger_tip.dae"/>
+        <mesh filename="package://robot_project/meshes/l_finger_tip.dae"/>
       </geometry>
     </visual>

File: urdf/head_camera.xacro (robot description, xacro)
@@ -25,5 +25,5 @@
       <inertia ixx="1e-6" ixy="0" ixz="0" iyy="1e-6" iyz="0" izz="1e-6" />
     </inertial>
-  </link>
+</link>
 <!--Σύνδεση κάμερας με το κεφάλι του ρομπότ με μία fixed άρθρωση-->
   <joint name="camera2_joint" type="fixed">

File: urdf/mantzakidisbot.xacro (robot description, xacro)
@@ -14,5 +14,5 @@
 <xacro:property name="w_mass" value="0.5" />           <!-- Μάζα των τροχών -->
  <!-- Εισαγωγή χρωμάτων Rviz -->
-  <xacro:include filename="$(find project_final_mantzakidis_131)/urdf/materials.xacro" />
+  <xacro:include filename="$(find robot_project)/urdf/materials.xacro" />
 <!-- Default Inertial -->
   <xacro:macro name="default_inertial" params="z_value i_value mass">
@@ -26,11 +26,11 @@
   </xacro:macro>
 <!-- Εισαγωγή URDF του βραχίονα -->
-  <xacro:include filename="$(find project_final_mantzakidis_131)/urdf/mantzakidisbot_arm.xacro" />
+  <xacro:include filename="$(find robot_project)/urdf/mantzakidisbot_arm.xacro" />
 <!-- Εισαγωγή στοιχείων Gazebo, συμπεριλαμβανομένων των χρωμάτων του Gazebo -->
-  <xacro:include filename="$(find project_final_mantzakidis_131)/urdf/mantzakidisbot.gazebo" />
+  <xacro:include filename="$(find robot_project)/urdf/mantzakidisbot.gazebo" />
 <!-- Εισαγωγή laser & camera-->
-  <xacro:include filename="$(find project_final_mantzakidis_131)/urdf/mantzakidisbot_laser_camera.xacro" />
+  <xacro:include filename="$(find robot_project)/urdf/mantzakidisbot_laser_camera.xacro" />
 <!-- Εισαγωγή κάμερας κεφαλιού-->
-  <xacro:include filename="$(find project_final_mantzakidis_131)/urdf/head_camera.xacro" />
+  <xacro:include filename="$(find robot_project)/urdf/head_camera.xacro" />
   <!-- Robot chassis -->
   <link name="chassis">
@@ -104,22 +104,22 @@
       </visual>
       <!-- Head collision, mass and inertia -->
-    <collision>
-      <origin xyz="0 0 0" rpy="0 0 0" />
-      <geometry>
-        <sphere radius="${head_radius}" />
-      </geometry>
-    </collision>
-    <inertial>
-      <mass value="${head_mass}"/>
-      <inertia ixx="0.004" ixy="0.0" ixz="0.0" iyy="0.004" iyz="0.0" izz="0.004"/>
-    </inertial>
+      <collision>
+        <origin xyz="0 0 0" rpy="0 0 0" />
+        <geometry>
+          <sphere radius="${head_radius}" />
+        </geometry>
+      </collision>
+      <inertial>
+        <mass value="${head_mass}"/>
+        <inertia ixx="0.004" ixy="0.0" ixz="0.0" iyy="0.004" iyz="0.0" izz="0.004"/>
+      </inertial>
     </link>
   <!--Head joint-->
-  <joint name="joint_head" type="continuous">
+  <joint name="joint_head" type="fixed">
     <parent link="chassis"/>
     <child link="head"/>
     <origin xyz="0 0 0.2" rpy="0 0 0" />
-    <axis xyz="0 0 1" />
-    <effort>joint_head_effort_interface</effort>
+    <!-- <axis xyz="0 0 1" /> -->
+    <!-- <effort>joint_head_effort_interface</effort> -->
   </joint>
 <!-- Right Wheel -->

File: urdf/mantzakidisbot_arm.xacro (robot description, xacro)
@@ -8,5 +8,5 @@
  <xacro:property name="damp" value="0.7" />  <!-- Aπόσβεση (damping) που εφαρμόζεται σε έναν αρθρωτό μηχανισμό για να μειωθούν οι δονήσεις-->
 <!-- Εισαγωγή URDF της αρπάγης -->
-  <xacro:include filename="$(find project_final_mantzakidis_131)/urdf/gripper.xacro" />
+  <xacro:include filename="$(find robot_project)/urdf/gripper.xacro" />
 <!-- Μακρο εντολή για τον υπολογισμό της αδράνειας-->
   <xacro:macro name="default_inertial" params="z_value i_value mass">

File: urdf/mantzakidisbot_laser_camera.xacro (robot description, xacro)
@@ -51,5 +51,5 @@
       <origin xyz="0 0 0" rpy="0 0 0"/>
       <geometry>
-        <mesh filename="package://project_final_mantzakidis_131/meshes/hokuyo.dae"/>
+        <mesh filename="package://robot_project/meshes/hokuyo.dae"/>
       </geometry>
     </visual>
