Commit message: added rviz

File: urdf/materials.xacro (robot description, xacro)
@@ -1,11 +1,11 @@
 <?xml version="1.0"?>
 <robot>
-<material name="black">
+  <material name="black">
     <color rgba="0 0 0 1"/>
   </material>
-<material name="green">
+  <material name="green">
     <color rgba="0 1 0 1"/>
   </material>
-<material name="red">
+  <material name="red">
     <color rgba="0.8 0.0 0.0 1.0"/>
   </material>
@@ -13,6 +13,27 @@
     <color rgba="0.0 0.0 0.8 1.0"/>
   </material>
- <material name="orange">
+  <material name="orange">
     <color rgba="${255/255} ${108/255} ${10/255} 1.0"/>
   </material>
+  <material name="yellow">
+    <color rgba="1.0 1.0 0.0 1.0"/>
+  </material>
+  <material name="purple">
+    <color rgba="0.5 0.0 0.5 1.0"/>
+  </material>
+  <material name="cyan">
+    <color rgba="0.0 1.0 1.0 1.0"/>
+  </material>
+  <material name="magenta">
+    <color rgba="1.0 0.0 1.0 1.0"/>
+  </material>
+  <material name="light_grey">
+    <color rgba="0.8 0.8 0.8 1.0"/>
+  </material>
+  <material name="dark_grey">
+    <color rgba="0.2 0.2 0.2 1.0"/>
+  </material>
+  <material name="gold">
+    <color rgba="${255/255} ${215/255} ${0/255} 1.0"/>
+  </material>
 </robot>
